Commit message: Created better garden. Also, isolate custom gazebo_worlds package.

File: src/hector_quadrotor-kinetic-devel/hector_quadrotor_description/urdf/quadrotor_with_kinect.urdf.xacro (robot description, xacro)
@@ -9,5 +9,5 @@
     <xacro:include filename="$(find hector_sensors_description)/urdf/kinect_camera.urdf.xacro" />
     <xacro:kinect_camera name="camera" parent="base_link">
-      <origin xyz="0.0 0.0 -0.1" rpy="0 ${M_PI/2} 0"/>
+      <origin xyz="0.0 0.0 -0.1" rpy="0 0 0"/>
     </xacro:kinect_camera>
 </robot>
